File: telex_interface.kicad_sch (KiCad schematic)
At the start: 43 parts, among them J1 DB25_Female_MountingHoles, J4 Raspberry_Pi_2_3, U1 max3387, U2 74LVC1G08

Commit message: moar work
Parts:
- removed J4: Raspberry_Pi_2_3, Connector_PinSocket_2.54mm:PinSocket_2x20_P2.54mm_Vertical, symbol Connector:Raspberry_Pi_2_3
- added J2: Conn_02x20_Odd_Even, Connector_PinSocket_2.54mm:PinSocket_2x20_P2.54mm_Vertical, symbol Connector_Generic:Conn_02x20_Odd_Even
- added JP10, JP8, JP9: SolderJumper_2_Bridged, Jumper:SolderJumper-2_P1.3mm_Bridged_Pad1.0x1.5mm, symbol Jumper:SolderJumper_2_Bridged
- added JP11, JP12, JP13: SolderJumper_2_Open, Jumper:SolderJumper-2_P1.3mm_Open_Pad1.0x1.5mm, symbol Jumper:SolderJumper_2_Open
- added TP20, TP21, TP22, TP23: TestPoint, TestPoint:TestPoint_Pad_2.0x2.0mm, symbol Connector:TestPoint
Connections:
- net GND: now also J2.14 (Pin_14), J2.20 (Pin_20), J2.25 (Pin_25), J2.30 (Pin_30), J2.34 (Pin_34), J2.39 (Pin_39), J2.6 (Pin_6), J2.9 (Pin_9), TP20.1, TP21.1
- net RxD_TTY: now also JP8.1 (A)
- net TxD: now also JP9.1 (A)
- net VCC: now also J2.1 (Pin_1), J2.17 (Pin_17)
- net ~{ARQ}: now also JP13.1 (A)
- net ~{BetrB_DTR}: now also JP12.1 (A)
- net ~{M2}: now also JP11.1 (A)
- net ~{S2_RTS}: now also JP10.1 (A)
- new net GPIO0_Tx3: J2.27 (Pin_27), TP22.1
- new net GPIO10: J2.19 (Pin_19), JP10.2 (B)
- new net GPIO11: J2.23 (Pin_23), JP13.2 (B)
- new net GPIO17: J2.11 (Pin_11), JP8.2 (B)
- new net GPIO1_Rx2: J2.28 (Pin_28), TP23.1
- new net GPIO22: J2.15 (Pin_15), JP12.2 (B)
- new net GPIO27: J2.13 (Pin_13), JP9.2 (B)
- new net GPIO9: J2.21 (Pin_21), JP11.2 (B)
- no-connect marks 40 -> 13
Other:
- note added: "ARQ (Req. Msg)"
- note added: "BetrB (On)"
- note added: "M2 (beep)"
- note added: "Raspberry Pi"
- note added: "RxD D2"
- note added: "S2 (Lin)"
- note added: "Teletype"
- note added: "TxD D1"
- note added: "V10"
- note added: "pin_observe_line"
- note added: "pin_rxd"
- note added: "pin_txd"
- note added: "telex.json"
- note removed: "Check Pins!!!"

Commit message: Further work...
Parts:
- removed TP22, TP23: TestPoint, TestPoint:TestPoint_Pad_2.0x2.0mm, symbol Connector:TestPoint
- added H1, H2: MountingHole, MountingHole:MountingHole_2.7mm_M2.5, symbol Mechanical:MountingHole
- added J3: Conn_01x03_Male, Connector_PinHeader_2.54mm:PinHeader_1x03_P2.54mm_Vertical, symbol Connector:Conn_01x03_Male
- added J4: Conn_02x04_Odd_Even, Connector_PinHeader_2.54mm:PinHeader_2x04_P2.54mm_Vertical, symbol Connector_Generic:Conn_02x04_Odd_Even
- added TP24, TP25, TP26: TestPoint, TestPoint:TestPoint_Pad_2.0x2.0mm, symbol Connector:TestPoint
Connections:
- net GND: now also J3.1 (Pin_1), J4.1 (Pin_1), J4.4 (Pin_4), TP26.1
- net V10_BetrB_DTR: now also U1.16 (R3in); no longer U1.18 (R1in)
- net V10_D1_TxD: now also U1.18 (R1in); no longer U1.16 (R3in)
- net VCC: now also J4.2 (Pin_2)
- net C1pos: now reaches C4.1, U1.1 (C1pos)
- net C1neg: now reaches C4.2, U1.3 (C1neg)
- net C2pos: now reaches C5.1, U1.4 (C2pos)
- net C2neg: now reaches C5.2, U1.5 (C2neg)
- net GPIO15_Cons_Rx: now reaches J2.10 (Pin_10)
- net GPIO15_Cons_Rx: now also J3.3 (Pin_3)
- net GPIO18_CE0: now reaches J2.12 (Pin_12)
- net GPIO18_CE0: now also J4.7 (Pin_7)
- net GPIO2_SDA: now reaches J2.3 (Pin_3)
- net GPIO2_SDA: now also TP25.1
- net GPIO19_CIPO: now reaches J2.35 (Pin_35)
- net GPIO19_CIPO: now also J4.5 (Pin_5)
- net GPIO16_CE2: now reaches J2.36 (Pin_36)
- net GPIO16_CE2: now also J4.8 (Pin_8)
- net GPIO20_COPI: now reaches J2.38 (Pin_38)
- net GPIO20_COPI: now also J4.6 (Pin_6)
- net GPIO21_SCLK: now reaches J2.40 (Pin_40)
- net GPIO21_SCLK: now also J4.3 (Pin_3)
- net GPIO3_SCL: now reaches J2.5 (Pin_5)
- net GPIO3_SCL: now also TP24.1
- net GPIO14_Cons_Tx: now reaches J2.8 (Pin_8)
- net GPIO14_Cons_Tx: now also J3.2 (Pin_2)
- net GPIO0_Tx3: no longer names the net of J2.27 (Pin_27)
- net GPIO1_Rx2: no longer names the net of J2.28 (Pin_28)
Other:
- note added: "74LVC1G08QSE-7 Diodes Incorporated SOT353 2.15mm x 2.1mm x 1.1mm 0.65mm pitch"
- note added: "Raspberry Pi Pin Header"
- note added: "Reichelt: D-SUB BU 25EU D-Sub Right Angle Type 9.4mm"
- note added: "Testpad/Solderpad 3.3V CMOS"
- note added: "Testpad/Solderpad Supply Voltages"
- note added: "Testpad/Solderpad V.10"
- moved on the sheet: C1, C2, C3, C4, C5, C6, C7, D1, J1, J2, JP1, JP10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
